File: STKbd.sch (EAGLE design)
At the start: 70 parts, among them IC1 MEGA8-AI, IC2 DS1813-SMD, Q1 20 MHz, X1 MKDSN1,5/2-5,08, X2 MKDSN1,5/2-5,08, X3 MKDSN1,5/2-5,08, X4 22-23-2021, X5 MKDSN1,5/2-5,08, X6 MKDSN1,5/2-5,08, X7 MKDSN1,5/2-5,08

Commit message: Rev 1.0
Parts:
- removed BTN1: SPST.B3U-1000P(M), omron:SPST.B3U-1000P(M)
- removed C13: (no value), rcl:CPOL-EU153CLV-0605
- removed C7, C8: (no value), rcl:C-EUC0805
- removed IC2: DS1813-SMD, ds1813_revised:DS1813-SMD
- removed LED10, LED11, LED6, LED7, LED8, LED9: LED, MyLib:LED
- removed R21: 1k, rcl:R-EU_R0805
- removed X4: 22-23-2021, con-molex:22-23-2021
- added C4: 0.1u, rcl:C-EUC0805K
- added C5, C6: (no value), rcl:C-EUC0805
- added D1, D10, D2, D3, D4, D5, D6, D7, D8, D9: BAV199, diode:BAV199
- added R22, R23, R24, R25, R26, R27: 50R, rcl:R-EU_R0805
- added U$10, U$7, U$8, U$9: NSI45020AT1GSOD-123, MyLib:NSI45020AT1GSOD-123
- added U$11: TRACO_TEL_3-2411, MyLib:TRACO_TEL_3-2411
- LED1: value (none) -> LED; device led:LEDCHIP-LED0805 -> MyLib:LED
- R10, R11, R7, R8, R9: value 50R -> 1k
- R16, R17, R18, R19: value 1k -> 50R
- R20: value 1k -> 10k
- X7: value MKDSN1,5/2-5,08 -> 22-23-2031; device con-phoenix-508:MKDSN1,5/2-5,08 -> con-molex:22-23-2031
Connections:
- removed net N$31 (its old number): LED9.A@1, R19.1
- removed net N$32 (its old number): LED10.A@1, R20.1
- removed net N$33 (its old number): LED11.A@1, R21.1
- removed net N$68: LED1.A, R1.1
- removed net N$76: IC1.ADC6
- new net N$17: D9.AC, R18.1, U$9.C
- new net N$18: R18.2, X6-1.KL
- new net N$19: D10.AC, R19.1, U$10.C
- new net N$20: R19.2, X6-2.KL
- new net N$34: OC1.EMIT, U$7.A
- new net N$38: D3.AC, R24.1, U$3.A
- new net N$39: D1.AC, R22.1, U$1.A
- new net N$40: D4.AC, R25.1, U$4.A
- new net N$41: D5.AC, R26.1, U$5.A
- new net N$42: D6.AC, R27.1, U$6.A
- new net N$43: R27.2, X3-1.KL
- new net N$44: LED1.A@1, R1.2
- net +24V: now also C5.1, C6.1, D1.C, D10.C, D2.C, D3.C, D4.C, D5.C, D6.C, D7.C, D8.C, D9.C, U$11.+VIN@1, U$11.+VIN@2, X7-1.S; no longer X7-1.KL
- net +5V: now also R1.1, R10.2, R11.2, R20.2, R6.2, R7.2, R8.2, R9.2, U$11.+VOUT@1, U$11.+VOUT@2; no longer C13.+, C7.1, C8.1, IC2.+5V, OC10.COL, OC5.COL, OC6.COL, OC7.COL, OC8.COL, OC9.COL, R1.2, X4-1.S
- net GND: now also C4.2, LED1.C@2, OC10.EMIT, OC5.EMIT, OC6.EMIT, OC7.EMIT, OC8.EMIT, OC9.EMIT, U$11.-V0UT@1, U$11.-V0UT@2; no longer BTN1.2, C13.-, C7.2, C8.2, IC2.GND, LED1.C, LED10.C@2, LED11.C@2, LED6.C@2, LED7.C@2, LED8.C@2, LED9.C@2, R10.1, R11.1, R6.1, R7.1, R8.1, R9.1, X4-2.S
- net K1: now also OC5.COL, R6.1; no longer OC5.EMIT, R16.2, R6.2
- net K2: now also OC6.COL, R7.1; no longer OC6.EMIT, R17.2, R7.2
- net K3: now also OC7.COL, R8.1; no longer OC7.EMIT, R18.2, R8.2
- net K4: now also OC8.COL, R9.1; no longer OC8.EMIT, R19.2, R9.2
- net N$10: now also D7.AC, R16.1, U$7.C; no longer OC1.EMIT, X5-1.KL
- net N$11: now also D8.AC, R17.1, U$8.C; no longer OC2.EMIT, X5-2.KL
- net N$13: now also R16.2, X5-1.KL; no longer OC3.EMIT, X6-2.KL
- net N$14: now also R17.2, X5-2.KL; no longer OC4.EMIT, X6-1.KL
- net N$22: now also R22.2; no longer U$2.A
- net N$24: now also R26.2, X3-2.KL; no longer U$4.A, X2-2.KL
- net N$25: now also R23.2, X1-1.KL; no longer U$5.A, X3-1.KL
- net N$26: now also R25.2, X2-1.KL; no longer U$6.A, X3-2.KL
- net N$28: now also OC4.EMIT, U$10.A; no longer LED6.A@1, R16.1
- net N$29: now also OC3.EMIT, U$9.A; no longer LED7.A@1, R17.1
- net N$30: now also OC2.EMIT, U$8.A; no longer LED8.A@1, R18.1
- net N$8: now also R24.2, X2-2.KL; no longer U$3.A, X2-1.KL
- net N$9: now also D2.AC, R23.1, U$2.A; no longer U$1.A, X1-1.KL
- net PE: now also C5.2, C6.2, D1.A, D10.A, D2.A, D3.A, D4.A, D5.A, D6.A, D7.A, D8.A, D9.A, U$11.-VIN@1, U$11.-VIN@2, X7-3.S; no longer X7-2.KL
- net RESET: now also C4.1, R20.1; no longer BTN1.1, IC2./RST
- net RS1: now also OC9.COL, R10.1; no longer OC9.EMIT, R10.2, R20.2
- net RS2: now also OC10.COL, R11.1; no longer OC10.EMIT, R11.2, R21.2
Other:
- moved on the sheet: LED1, LED2, LED3, LED4, LED5, OC1, OC10, OC2, OC3, OC4, OC5, OC7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

Commit message: rev 1.1 to produce
Connections:
- removed net S4: IC1.PC3(ADC3), R15.1, R5.1
- new net S44: IC1.PC0(ADC0), R12.1, R2.1
- net K1: now also IC1.PD7(AIN1), OC10.COL, R11.1; no longer IC1.PD4(XCK/T0), OC5.COL, R6.1
- net K2: now also IC1.PD6(AIN0), OC9.COL, R10.1; no longer IC1.PD5(T1), OC6.COL, R7.1
- net K3: now also IC1.PD5(T1), OC8.COL, R9.1; no longer IC1.PD6(AIN0), OC7.COL, R8.1
- net K4: now also IC1.PD4(XCK/T0), OC7.COL, R8.1; no longer IC1.PD7(AIN1), OC8.COL, R9.1
- net RS1: now also IC1.PD3(INT1), OC6.COL, R7.1; no longer IC1.PD2(INT0), OC9.COL, R10.1
- net RS2: now also IC1.PD2(INT0), OC5.COL, R6.1; no longer IC1.PD3(INT1), OC10.COL, R11.1
- net S1: now also IC1.PC3(ADC3), R15.1, R5.1; no longer IC1.PC0(ADC0), R12.1, R2.1
- net S2: now also IC1.PC2(ADC2), R14.1, R4.1; no longer IC1.PC1(ADC1), R13.1, R3.1
- net S3: now also IC1.PC1(ADC1), R13.1, R3.1; no longer IC1.PC2(ADC2), R14.1, R4.1
Changed lines of the file:
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@@
-</segment>
-</net>
-<net name="RS1" class="0">
-<segment>
-<pinref part="IC1" gate="G$1" pin="PD2(INT0)"/>
-<label x="-55.88" y="15.24" size="1.778" layer="95"/>
-<wire x1="-60.96" y1="15.24" x2="-20.32" y2="15.24" width="0.1524" layer="91"/>
-<wire x1="-20.32" y1="15.24" x2="-20.32" y2="-99.06" width="0.1524" layer="91"/>
-<pinref part="OC9" gate="A" pin="COL"/>
-<pinref part="R10" gate="G$1" pin="1"/>
-<wire x1="2.54" y1="-99.06" x2="2.54" y2="-96.52" width="0.1524" layer="91"/>
-<wire x1="2.54" y1="-99.06" x2="-20.32" y2="-99.06" width="0.1524" layer="91"/>
-</segment>
-</net>
-<net name="RS2" class="0">
-<segment>
-<pinref part="IC1" gate="G$1" pin="PD3(INT1)"/>
-<label x="-55.88" y="12.7" size="1.778" layer="95"/>
-<wire x1="-22.86" y1="-127" x2="-22.86" y2="12.7" width="0.1524" layer="91"/>
-<wire x1="-22.86" y1="12.7" x2="-60.96" y2="12.7" width="0.1524" layer="91"/>
-<pinref part="OC10" gate="A" pin="COL"/>
-<pinref part="R11" gate="G$1" pin="1"/>
-<wire x1="2.54" y1="-124.46" x2="2.54" y2="-127" width="0.1524" layer="91"/>
-<wire x1="2.54" y1="-127" x2="-22.86" y2="-127" width="0.1524" layer="91"/>
-</segment>
-</net>
-<net name="K2" class="0">
-<segment>
-<pinref part="IC1" gate="G$1" pin="PD5(T1)"/>
-<label x="-55.88" y="7.62" size="1.778" layer="95"/>
-<wire x1="-12.7" y1="7.62" x2="-60.96" y2="7.62" width="0.1524" layer="91"/>
-<pinref part="R7" gate="G$1" pin="1"/>
-<pinref part="OC6" gate="A" pin="COL"/>
-<wire x1="2.54" y1="-15.24" x2="2.54" y2="-17.78" width="0.1524" layer="91"/>
-<wire x1="-12.7" y1="7.62" x2="-12.7" y2="-17.78" width="0.1524" layer="91"/>
-<wire x1="-12.7" y1="-17.78" x2="2.54" y2="-17.78" width="0.1524" layer="91"/>
-</segment>
-</net>
-<net name="K3" class="0">
-<segment>
-<pinref part="IC1" gate="G$1" pin="PD6(AIN0)"/>
-<label x="-55.88" y="5.08" size="1.778" layer="95"/>
-<wire x1="-60.96" y1="5.08" x2="-15.24" y2="5.08" width="0.1524" layer="91"/>
-<wire x1="-15.24" y1="5.08" x2="-15.24" y2="-43.18" width="0.1524" layer="91"/>
-<pinref part="R8" gate="G$1" pin="1"/>
-<pinref part="OC7" gate="A" pin="COL"/>
-<wire x1="2.54" y1="-40.64" x2="2.54" y2="-43.18" width="0.1524" layer="91"/>
-<wire x1="-15.24" y1="-43.18" x2="2.54" y2="-43.18" width="0.1524" layer="91"/>
-</segment>
-</net>
-<net name="K4" class="0">
-<segment>
-<pinref part="IC1" gate="G$1" pin="PD7(AIN1)"/>
-<label x="-55.88" y="2.54" size="1.778" layer="95"/>
-<wire x1="-17.78" y1="-71.12" x2="-17.78" y2="2.54" width="0.1524" layer="91"/>
-<wire x1="-17.78" y1="2.54" x2="-60.96" y2="2.54" width="0.1524" layer="91"/>
-<pinref part="OC8" gate="A" pin="COL"/>
-<pinref part="R9" gate="G$1" pin="1"/>
-<wire x1="2.54" y1="-68.58" x2="2.54" y2="-71.12" width="0.1524" layer="91"/>
-<wire x1="2.54" y1="-71.12" x2="-17.78" y2="-71.12" width="0.1524" layer="91"/>
 </segment>
 </net>
@@
 </segment>
 </net>
-<net name="K1" class="0">
-<segment>
-<pinref part="IC1" gate="G$1" pin="PD4(XCK/T0)"/>
-<wire x1="-60.96" y1="10.16" x2="2.54" y2="10.16" width="0.1524" layer="91"/>
-<label x="-55.88" y="10.16" size="1.778" layer="95"/>
+<net name="RS2" class="0">
+<segment>
 <pinref part="OC5" gate="A" pin="COL"/>
 <pinref part="R6" gate="G$1" pin="1"/>
-</segment>
-</net>
-<net name="S1" class="0">
+<pinref part="IC1" gate="G$1" pin="PD2(INT0)"/>
+<wire x1="-60.96" y1="15.24" x2="-10.16" y2="15.24" width="0.1524" layer="91"/>
+<wire x1="-10.16" y1="15.24" x2="-10.16" y2="10.16" width="0.1524" layer="91"/>
+<wire x1="-10.16" y1="10.16" x2="2.54" y2="10.16" width="0.1524" layer="91"/>
+<label x="-17.78" y="15.24" size="1.778" layer="95"/>
+</segment>
+</net>
+<net name="S44" class="0">
 <segment>
 <pinref part="R2" gate="G$1" pin="1"/>
@@
 </segment>
 </net>
-<net name="S2" class="0">
+<net name="S3" class="0">
 <segment>
 <pinref part="IC1" gate="G$1" pin="PC1(ADC1)"/>
@@
 </segment>
 </net>
-<net name="S3" class="0">
+<net name="S2" class="0">
 <segment>
 <pinref part="IC1" gate="G$1" pin="PC2(ADC2)"/>
@@
 </segment>
 </net>
-<net name="S4" class="0">
+<net name="S1" class="0">
 <segment>
 <pinref part="IC1" gate="G$1" pin="PC3(ADC3)"/>
@@
 </segment>
 </net>
+<net name="K2" class="0">
+<segment>
+<pinref part="R10" gate="G$1" pin="1"/>
+<pinref part="OC9" gate="A" pin="COL"/>
+<wire x1="2.54" y1="-99.06" x2="2.54" y2="-96.52" width="0.1524" layer="91"/>
+<pinref part="IC1" gate="G$1" pin="PD6(AIN0)"/>
+<wire x1="-60.96" y1="5.08" x2="-20.32" y2="5.08" width="0.1524" layer="91"/>
+<wire x1="-20.32" y1="5.08" x2="-20.32" y2="-99.06" width="0.1524" layer="91"/>
+<wire x1="-20.32" y1="-99.06" x2="2.54" y2="-99.06" width="0.1524" layer="91"/>
+<label x="-20.32" y="-93.98" size="1.778" layer="95"/>
+</segment>
+</net>
+<net name="RS1" class="0">
+<segment>
+<pinref part="OC6" gate="A" pin="COL"/>
+<pinref part="R7" gate="G$1" pin="1"/>
+<wire x1="2.54" y1="-15.24" x2="2.54" y2="-17.78" width="0.1524" layer="91"/>
+<pinref part="IC1" gate="G$1" pin="PD3(INT1)"/>
+<wire x1="-60.96" y1="12.7" x2="-12.7" y2="12.7" width="0.1524" layer="91"/>
+<wire x1="-12.7" y1="12.7" x2="-12.7" y2="-17.78" width="0.1524" layer="91"/>
+<wire x1="-12.7" y1="-17.78" x2="2.54" y2="-17.78" width="0.1524" layer="91"/>
+<label x="-12.7" y="-7.62" size="1.778" layer="95"/>
+</segment>
+</net>
+<net name="K4" class="0">
+<segment>
+<pinref part="OC7" gate="A" pin="COL"/>
+<pinref part="R8" gate="G$1" pin="1"/>
+<wire x1="2.54" y1="-40.64" x2="2.54" y2="-43.18" width="0.1524" layer="91"/>
+<pinref part="IC1" gate="G$1" pin="PD4(XCK/T0)"/>
+<wire x1="-60.96" y1="10.16" x2="-15.24" y2="10.16" width="0.1524" layer="91"/>
+<wire x1="-15.24" y1="10.16" x2="-15.24" y2="-43.18" width="0.1524" layer="91"/>
+<wire x1="-15.24" y1="-43.18" x2="2.54" y2="-43.18" width="0.1524" layer="91"/>
+<label x="-15.24" y="-35.56" size="1.778" layer="95"/>
+</segment>
+</net>
+<net name="K3" class="0">
+<segment>
+<pinref part="OC8" gate="A" pin="COL"/>
+<pinref part="R9" gate="G$1" pin="1"/>
+<wire x1="2.54" y1="-68.58" x2="2.54" y2="-71.12" width="0.1524" layer="91"/>
+<pinref part="IC1" gate="G$1" pin="PD5(T1)"/>
+<wire x1="-60.96" y1="7.62" x2="-17.78" y2="7.62" width="0.1524" layer="91"/>
+<wire x1="-17.78" y1="7.62" x2="-17.78" y2="-71.12" width="0.1524" layer="91"/>
+<wire x1="-17.78" y1="-71.12" x2="2.54" y2="-71.12" width="0.1524" layer="91"/>
+<label x="-17.78" y="-60.96" size="1.778" layer="95"/>
+</segment>
+</net>
+<net name="K1" class="0">
+<segment>
+<pinref part="OC10" gate="A" pin="COL"/>
+<wire x1="2.54" y1="-127" x2="-22.86" y2="-127" width="0.1524" layer="91"/>
+<pinref part="R11" gate="G$1" pin="1"/>
+<wire x1="2.54" y1="-124.46" x2="2.54" y2="-127" width="0.1524" layer="91"/>
+<pinref part="IC1" gate="G$1" pin="PD7(AIN1)"/>
+<wire x1="-60.96" y1="2.54" x2="-22.86" y2="2.54" width="0.1524" layer="91"/>
+<wire x1="-22.86" y1="2.54" x2="-22.86" y2="-127" width="0.1524" layer="91"/>
+<label x="-22.86" y="-114.3" size="1.778" layer="95"/>
+</segment>
+</net>

Commit message: rev 1.2 to produce
Parts:
- removed C9: (no value), rcl:C-EUC0805
- added JP2: (no value), pinhead:PINHD-1X2
- added JP3: (no value), pinhead:PINHD-1X3
Connections:
- net +5V: no longer C9.1
- net GND: now also JP3.1; no longer C9.2
- net RXD: now also JP2.1
- net SCL: now also JP3.3
- net SDA: now also JP3.2
- net TXD: now also JP2.2
Changed lines of the file:
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@@
 <part name="GND24" library="supply1" deviceset="GND" device=""/>
 <part name="P+6" library="supply1" deviceset="+5V" device=""/>
-<part name="C9" library="rcl" deviceset="C-EU" device="C0805"/>
 <part name="C10" library="rcl" deviceset="C-EU" device="C0805"/>
 <part name="C11" library="rcl" deviceset="C-EU" device="C0805"/>
@@
 <part name="C5" library="rcl" deviceset="C-EU" device="C0805"/>
 <part name="C6" library="rcl" deviceset="C-EU" device="C0805"/>
+<part name="JP2" library="pinhead" deviceset="PINHD-1X2" device=""/>
+<part name="JP3" library="pinhead" deviceset="PINHD-1X3" device=""/>
+<part name="GND1" library="supply1" deviceset="GND" device=""/>
 </parts>
 <sheets>
@@
 <instance part="GND24" gate="1" x="-147.32" y="-63.5"/>
 <instance part="P+6" gate="1" x="-147.32" y="-50.8"/>
-<instance part="C9" gate="G$1" x="-160.02" y="-55.88"/>
 <instance part="C10" gate="G$1" x="-167.64" y="-55.88"/>
 <instance part="C11" gate="G$1" x="-177.8" y="-55.88"/>
@@
 <instance part="C5" gate="G$1" x="-261.62" y="-60.96"/>
 <instance part="C6" gate="G$1" x="-251.46" y="-60.96"/>
+<instance part="JP2" gate="G$1" x="-30.48" y="20.32"/>
+<instance part="JP3" gate="A" x="-43.18" y="-38.1"/>
+<instance part="GND1" gate="1" x="-73.66" y="-38.1"/>
 </instances>
 <busses>
@@
 <wire x1="-187.96" y1="-60.96" x2="-177.8" y2="-60.96" width="0.1524" layer="91"/>
 <wire x1="-177.8" y1="-60.96" x2="-167.64" y2="-60.96" width="0.1524" layer="91"/>
-<wire x1="-167.64" y1="-60.96" x2="-160.02" y2="-60.96" width="0.1524" layer="91"/>
-<pinref part="C9" gate="G$1" pin="2"/>
-<junction x="-160.02" y="-60.96"/>
 <pinref part="C10" gate="G$1" pin="2"/>
 <junction x="-167.64" y="-60.96"/>
@@
 <junction x="-177.8" y="-60.96"/>
 <junction x="-187.96" y="-60.96"/>
-<wire x1="-160.02" y1="-60.96" x2="-147.32" y2="-60.96" width="0.1524" layer="91"/>
+<wire x1="-167.64" y1="-60.96" x2="-147.32" y2="-60.96" width="0.1524" layer="91"/>
 <pinref part="U$11" gate="G$1" pin="-V0UT@1"/>
 <pinref part="U$11" gate="G$1" pin="-V0UT@2"/>
@@
 <pinref part="C4" gate="G$1" pin="2"/>
 <pinref part="GND17" gate="1" pin="GND"/>
+</segment>
+<segment>
+<pinref part="JP3" gate="A" pin="1"/>
+<wire x1="-45.72" y1="-35.56" x2="-73.66" y2="-35.56" width="0.1524" layer="91"/>
+<pinref part="GND1" gate="1" pin="GND"/>
 </segment>
 </net>
@@
 <pinref part="C10" gate="G$1" pin="1"/>
 <junction x="-167.64" y="-53.34"/>
-<wire x1="-167.64" y1="-53.34" x2="-160.02" y2="-53.34" width="0.1524" layer="91"/>
-<pinref part="C9" gate="G$1" pin="1"/>
-<junction x="-160.02" y="-53.34"/>
-<wire x1="-160.02" y1="-53.34" x2="-147.32" y2="-53.34" width="0.1524" layer="91"/>
+<wire x1="-167.64" y1="-53.34" x2="-147.32" y2="-53.34" width="0.1524" layer="91"/>
 <pinref part="U$11" gate="G$1" pin="+VOUT@1"/>
 <wire x1="-187.96" y1="-53.34" x2="-208.28" y2="-53.34" width="0.1524" layer="91"/>
@@
 <segment>
 <pinref part="IC1" gate="G$1" pin="PC4(ADC4/SDA)"/>
-<wire x1="-60.96" y1="33.02" x2="-43.18" y2="33.02" width="0.1524" layer="91"/>
+<wire x1="-60.96" y1="33.02" x2="-33.02" y2="33.02" width="0.1524" layer="91"/>
 <label x="-50.8" y="33.02" size="1.778" layer="95"/>
 </segment>
+<segment>
+<pinref part="JP3" gate="A" pin="2"/>
+<wire x1="-45.72" y1="-38.1" x2="-63.5" y2="-38.1" width="0.1524" layer="91"/>
+<label x="-58.42" y="-38.1" size="1.778" layer="95"/>
+</segment>
 </net>
 <net name="SCL" class="0">
 <segment>
 <pinref part="IC1" gate="G$1" pin="PC5(ADC5/SCL)"/>
-<wire x1="-60.96" y1="30.48" x2="-43.18" y2="30.48" width="0.1524" layer="91"/>
+<wire x1="-60.96" y1="30.48" x2="-33.02" y2="30.48" width="0.1524" layer="91"/>
 <label x="-50.8" y="30.48" size="1.778" layer="95"/>
+</segment>
+<segment>
+<pinref part="JP3" gate="A" pin="3"/>
+<wire x1="-45.72" y1="-40.64" x2="-63.5" y2="-40.64" width="0.1524" layer="91"/>
+<label x="-58.42" y="-40.64" size="1.778" layer="95"/>
 </segment>
 </net>
@@
 <segment>
 <pinref part="IC1" gate="G$1" pin="PD0(RXD)"/>
-<wire x1="-60.96" y1="20.32" x2="-53.34" y2="20.32" width="0.1524" layer="91"/>
+<wire x1="-60.96" y1="20.32" x2="-50.8" y2="20.32" width="0.1524" layer="91"/>
 <label x="-55.88" y="20.32" size="1.778" layer="95"/>
+<wire x1="-50.8" y1="20.32" x2="-50.8" y2="22.86" width="0.1524" layer="91"/>
+<pinref part="JP2" gate="G$1" pin="1"/>
+<wire x1="-50.8" y1="22.86" x2="-33.02" y2="22.86" width="0.1524" layer="91"/>
 </segment>
 </net>
@@
 <segment>
 <pinref part="IC1" gate="G$1" pin="PD1(TXD)"/>
-<wire x1="-60.96" y1="17.78" x2="-53.34" y2="17.78" width="0.1524" layer="91"/>
+<wire x1="-60.96" y1="17.78" x2="-48.26" y2="17.78" width="0.1524" layer="91"/>
 <label x="-55.88" y="17.78" size="1.778" layer="95"/>
-</segment>
-</net>
+<pinref part="JP2" gate="G$1" pin="2"/>
+<wire x1="-33.02" y1="20.32" x2="-48.26" y2="20.32" width="0.1524" layer="91"/>
+<wire x1="-48.26" y1="20.32" x2="-48.26" y2="17.78" width="0.1524" layer="91"/>
+</segment>
+</net>

Commit message: rev 1.3 to produce
Connections:
- net S44 renamed S4
Changed lines of the file:
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@@
 </segment>
 </net>
-<net name="S44" class="0">
+<net name="S4" class="0">
 <segment>
 <pinref part="R2" gate="G$1" pin="1"/>
